File: {{cookiecutter.project_name}}/hardware/{{cookiecutter.project_name}}.kicad_pcb (KiCad board)
At the start: 2 copper layers, 0 parts

Commit message: testing
Parts:
- added G***: LOGO, LOGO, F.Cu at (160.9, 121.7)
Other:
- board outline added: 50 x 50 mm
- copper layers 2 -> 4
- board text added: "0"
- board text added: "0 mm"
- board text added: "0,01 mm"
- board text added: "0,02"
- board text added: "0,035 mm"
- board text added: "0,1 mm"
- board text added: "0,1270 mm / 0,2540 mm"
- board text added: "0,2000 mm"
- board text added: "1"
- board text added: "1,24 mm"
- board text added: "1,6000 mm"
- board text added: "3,3"
- board text added: "4"
- board text added: "4,5"
- board text added: "50,0000 mm x 50,0000 mm"
- board text added: "62F B97A 71E9"
- board text added: "B.Cu"
- board text added: "B.Mask"
- board text added: "B.Paste"
- board text added: "B.Silkscreen"
- board text added: "BOARD CHARACTERISTICS"
- board text added: "Board Thickness:"
- board text added: "Board overall dimensions:"
- board text added: "Bottom Silk Screen"
- board text added: "Bottom Solder Mask"
- board text added: "Bottom Solder Paste"
- board text added: "Castellated pads:"
- board text added: "Color"
- board text added: "Copper Finish:"
- board text added: "Copper Layer Count:"
- board text added: "Dielectric 1"
- board text added: "Dielectric 2"
- board text added: "Dielectric 3"
- board text added: "ENIG"
- board text added: "Edge card connectors:"
- board text added: "Epsilon R"
- board text added: "F.Cu"
- board text added: "F.Mask"
- board text added: "F.Paste"
- board text added: "F.Silkscreen"
- board text added: "FR4"
- board text added: "Impedance Control:"
- board text added: "In1.Cu"
- board text added: "In2.Cu"
- board text added: "Layer Name"
- board text added: "Loss Tangent"
- board text added: "Magic Number Please Place Somewhere"
- board text added: "Material"
- board text added: "Min hole diameter:"
- board text added: "Min track/spacing:"
- board text added: "No"
- board text added: "Not specified"
- board text added: "Plated Board Edge:"
- board text added: "Thickness (mm)"
- board text added: "Top Silk Screen"
- board text added: "Top Solder Mask"
- board text added: "Top Solder Paste"
- board text added: "Type"
- board text added: "Yes"
- board text added: "copper"
- board text added: "core"
- board text added: "prepreg"
