File: {{cookiecutter.project_name}}/hardware/{{cookiecutter.project_name}}.kicad_sch (KiCad schematic)
At the start: 0 parts

Commit message: added department
Other:
- company: (none) -> IoT.nxt
Changed lines of the file:
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@@
     (date "{% now 'utc', '%Y-%m-%d' %}")
     (rev "A")
+    (company "IoT.nxt")
     (comment 1 "Author: {{cookiecutter.author_name}}")
     (comment 2 "Project Github: https://github.com/{{cookiecutter.github_user}}/{{cookiecutter.project_repo_name}}")
-    (comment 3 "License: {{cookiecutter.license}}")
+    (comment 3 "Department: {{cookiecutter.department}}")
   )
   (sheet_instances

Commit message: testing
Other:
- title: {{cookiecutter.project_description}} -> {{cookiecutter.project_name}}
Changed lines of the file:
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@@
   (paper "A4")
   (title_block
-    (title "{{cookiecutter.project_description}}")
+    (title "{{cookiecutter.project_name}}")
     (date "{% now 'utc', '%Y-%m-%d' %}")
     (rev "A")
     (company "IoT.nxt")
     (comment 1 "Author: {{cookiecutter.author_name}}")
-    (comment 2 "Project Github: https://github.com/{{cookiecutter.github_user}}/{{cookiecutter.project_repo_name}}")
-    (comment 3 "Department: {{cookiecutter.department}}")
+    (comment 2 "Department: {{cookiecutter.department}}")
   )
   (sheet_instances
